Commit message: Add robotiq sander

File: fanuc_description/urdf/fanuc.urdf (robot description, URDF)
Before this commit: robot fanuc, 9 links, 8 joints
Links:
- link tool0: geometry collision mesh filename=package://moveit_resources_fanuc_description/meshes/collisi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 scale=0.001 0.001 0.001; visual mesh filename=package://moveit_resources_fanuc_description/meshes/visual/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 scale=0.001 0.001 0.001
Joints:
- joint joint_6-tool0: origin xyz=0 0 0 rpy=3.1415926535 -1.570796327 0 -> xyz=0.1 0 0 rpy=3.1415926535 -1.570796327 0
